File: driver/driver.kicad_pcb (KiCad board)
At the start: 2 copper layers, 0 parts

Commit message: changed to correct RJ45-Plug
Parts:
- added C1: 0.1uF, Capacitor_SMD:C_0603_1608Metric_Pad1.05x0.95mm_HandSolder, F.Cu at (56.0, 60.0)
- added J1: signal_in, Connector_PinHeader_2.54mm:PinHeader_1x06_P2.54mm_Horizontal, B.Cu at (52.0, 66.3)
- added J2: LVDS_output, Connector_RJ:RJ45_Stewart_SS-6488S-A-NF, F.Cu at (78.0, 60.0)
- added R1: 10k, Resistor_SMD:R_1206_3216Metric_Pad1.42x1.75mm_HandSolder, F.Cu at (60.0, 67.0)
- added U1: SN65LVDS391, Package_SO:SOIC-16_3.9x9.9mm_P1.27mm, F.Cu at (62.0, 60.0)
Other:
- board outline added: 32 x 20 mm

Commit message: Driver finalized
Parts:
- moved R1 13.8 mm to (60.8, 53.2)
Connections:
- J1 pad 1: +3V3 -> GND
- J1 pad 2: /signal1 -> /signal3
- J1 pad 4: /signal3 -> /signal1
- J1 pad 6: GND -> +3V3
Routing:
- net +3V3: track 0.00 -> 16.8 mm, vias 0 -> 2
- net Net-(J2-PadSH): track 0.00 -> 15.5 mm
- net /EN: track 0.00 -> 14.9 mm
- net GND: track 0.00 -> 14.0 mm, vias 0 -> 1
- net /pair2-: track 0.00 -> 9.69 mm
- net /pair4-: track 0.00 -> 9.39 mm
- net /pair1+: track 0.00 -> 8.86 mm
- net /signal2: track 0.00 -> 7.85 mm
- net /signal1: track 0.00 -> 7.85 mm
- net /signal4: track 0.00 -> 7.56 mm
- net /signal3: track 0.00 -> 7.56 mm
- net /pair2+: track 0.00 -> 7.48 mm
- net /pair3-: track 0.00 -> 6.95 mm
- net /pair4+: track 0.00 -> 4.94 mm
- net /pair1-: track 0.00 -> 4.94 mm
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- added copper zone on B.Cu, net GND
- added copper zone on F.Cu, net GND
Other:
- board text added: "+3V3"
- board text added: "+3V3 S4 S1 S2 S3 GND"
- board text added: "DRIVER"
- board text added: "GND"
- board text added: "IN"
- board text added: "S1"
- board text added: "S2"
- board text added: "S3"
- board text added: "S4"
- board text added: "github.com/s-light/lvds_4ch_link"
- board text added: "v0.1.0 13.12.2018 cc by Stefan Krüger"
