File: receiver/receiver.sch (KiCad schematic (older format))
At the start: 0 parts

Commit message: prepaired link
Parts:
- added C? (x2): 0.1uF, Capacitor_SMD:C_0603_1608Metric_Pad1.05x0.95mm_HandSolder, symbol Device:C
- added J?: LVDS_input, symbol Connector:8P8C_Shielded
- added J?: LVDS_output, symbol Connector:8P8C_Shielded
- added J?: signal_in, symbol Connector_Generic:Conn_01x06
- added J?: signal_out, symbol Connector_Generic:Conn_01x06
- added U?: SN65LVDS391, Package_SO:SOIC-16_3.9x9.9mm_P1.27mm, symbol Interface:SN65LVDS391
- added U?: SN65LVDT348, Package_SO:SOIC-16_3.9x9.9mm_P1.27mm, symbol Interface:SN65LVDT348
Connections:
- new net +3V3: C?.1, C?.1, J?.1 (Pin_1), J?.1 (Pin_1), U?.13 (VCC), U?.4 (VCC)
- new net EN: U?.1 (EN1,2), U?.16 (EN), U?.8 (EN3,4)
- new net GND: C?.2, C?.2, J?.6 (Pin_6), J?.6 (Pin_6), U?.12 (GND), U?.5 (GND)
- new net pair1+: J?.5, J?.5, U?.14 (2Y), U?.3 (RIN2+)
- new net pair1-: J?.4, J?.4, U?.13 (2Z), U?.4 (RIN2-)
- new net pair2+: J?.3, J?.3, U?.12 (3Y), U?.6 (RIN3+)
- new net pair2-: J?.6, J?.6, U?.11 (3Z), U?.5 (RIN3-)
- new net pair3+: J?.2, J?.2, U?.10 (4Y), U?.7 (RIN4+)
- new net pair3-: J?.1, J?.1, U?.8 (RIN4-), U?.9 (4Z)
- new net pair4+: J?.8, J?.8, U?.15 (1Y), U?.2 (RIN1+)
- new net pair4-: J?.7, J?.7, U?.1 (RIN1-), U?.16 (1Z)
- new net signal1: J?.2 (Pin_2), J?.2 (Pin_2), U?.14 (ROUT2), U?.3 (2A)
- new net signal2: J?.3 (Pin_3), J?.3 (Pin_3), U?.11 (ROUT3), U?.6 (3A)
- new net signal3: J?.4 (Pin_4), J?.4 (Pin_4), U?.10 (ROUT4), U?.7 (4A)
- new net signal4: J?.5 (Pin_5), J?.5 (Pin_5), U?.15 (ROUT1), U?.2 (1A)
- no-connect marks 0 -> 3
Other:
- note added: "1 pair3- w/green\n2 pair3+ green\n3 pair2+ w/orange\n4 pair1- blue\n5 pair1+ w/blue\n6 pair2- orange\n7 pair4- w/brown\n8 pair4+ brown"
- note added: "8 pair4+ brown\n7 pair4- w/brown\n6 pair2- orange\n5 pair1+ w/blue\n4 pair1- blue\n3 pair2+ w/orange\n2 pair3+ green\n1 pair3- w/green"

Commit message: basic placement + added pullup for EN
Parts:
- removed C?: 0.1uF, Capacitor_SMD:C_0603_1608Metric_Pad1.05x0.95mm_HandSolder, symbol Device:C
- removed J?: LVDS_output, symbol Connector:8P8C_Shielded
- removed J?: signal_in, symbol Connector_Generic:Conn_01x06
- removed U?: SN65LVDS391, Package_SO:SOIC-16_3.9x9.9mm_P1.27mm, symbol Interface:SN65LVDS391
- added R1: 10k, Resistor_SMD:R_1206_3216Metric_Pad1.42x1.75mm_HandSolder, symbol Device:R
- J1: renamed from J?; footprint (none) -> Connector_RJ:RJ45_Amphenol_RJHSE5380
- J2: renamed from J?; footprint (none) -> Connector_PinHeader_2.54mm:PinHeader_1x06_P2.54mm_Horizontal
- gave numbers to parts that had none: 2
Connections:
- net +3V3: now also R1.1
- net EN: now also R1.2
- no-connect marks 3 -> 2
Changed lines of the file:
@@
 EESchema Schematic File Version 4
+LIBS:receiver-cache
 EELAYER 29 0
 EELAYER END
@@
 $EndDescr
 $Comp
-L Interface:SN65LVDS391 U?
-U 1 1 5C13291D
-P 2600 2300
-F 0 "U?" H 2350 3050 50  0000 C CNN
-F 1 "SN65LVDS391" H 2900 3050 50  0000 C CNN
-F 2 "Package_SO:SOIC-16_3.9x9.9mm_P1.27mm" H 2600 1550 50  0001 C CNN
-F 3 "http://www.ti.com/lit/ds/symlink/sn65lvds391.pdf" H 2600 2100 50  0001 C CNN
-	1    2600 2300
-	1    0    0    -1
-$EndComp
-$Comp
-L Interface:SN65LVDT348 U?
+L Interface:SN65LVDT348 U1
 U 1 1 5C14F4D9
 P 7600 2300
-F 0 "U?" H 7150 3150 50  0000 C CNN
+F 0 "U1" H 7150 3150 50  0000 C CNN
 F 1 "SN65LVDT348" H 7900 3150 50  0000 C CNN
 F 2 "Package_SO:SOIC-16_3.9x9.9mm_P1.27mm" H 7700 1400 50  0001 C CNN
@@
 $EndComp
 $Comp
-L Connector:8P8C_Shielded J?
+L Connector:8P8C_Shielded J1
 U 1 1 5C15786C
 P 5800 2500
-F 0 "J?" H 5857 3167 50  0000 C CNN
+F 0 "J1" H 5857 3167 50  0000 C CNN
 F 1 "LVDS_input" H 5857 3076 50  0000 C CNN
-F 2 "" V 5800 2525 50  0001 C CNN
+F 2 "Connector_RJ:RJ45_Amphenol_RJHSE5380" V 5800 2525 50  0001 C CNN
 F 3 "~" V 5800 2525 50  0001 C CNN
 	1    5800 2500
 	1    0    0    -1
 $EndComp
-$Comp
-L Connector:8P8C_Shielded J?
-U 1 1 5C15839B
-P 4200 2500
-F 0 "J?" H 4250 3150 50  0000 R CNN
-F 1 "LVDS_output" H 4350 3050 50  0000 R CNN
-F 2 "" V 4200 2525 50  0001 C CNN
-F 3 "~" V 4200 2525 50  0001 C CNN
-	1    4200 2500
-	-1   0    0    -1
-$EndComp
 Text Notes 4650 1800 0    50   ~ 0
 1 pair3-  w/green\n2 pair3+ green\n3 pair2+ w/orange\n4 pair1- blue\n5 pair1+ w/blue\n6 pair2- orange\n7 pair4-  w/brown\n8 pair4+ brown
-Text Label 3800 2800 2    50   ~ 0
-pair3-
-Text Label 3800 2700 2    50   ~ 0
-pair3+
 Text Notes 4600 2700 0    50   ~ 0
 8 pair4+ brown\n7 pair4-  w/brown\n6 pair2- orange\n5 pair1+ w/blue\n4 pair1- blue\n3 pair2+ w/orange\n2 pair3+ green\n1 pair3-  w/green
-Text Label 3800 2300 2    50   ~ 0
-pair2-
-Text Label 3800 2600 2    50   ~ 0
-pair2+
-Text Label 3800 2500 2    50   ~ 0
-pair1-
-Text Label 3800 2400 2    50   ~ 0
-pair1+
-Text Label 3800 2200 2    50   ~ 0
-pair4-
-Text Label 3800 2100 2    50   ~ 0
-pair4+
 Text Label 6200 2800 0    50   ~ 0
 pair3-
@@
 pair4-
 Text Label 6200 2100 0    50   ~ 0
-pair4+
-Text Label 2200 1800 2    50   ~ 0
-signal4
-Text Label 2200 2800 2    50   ~ 0
-signal3
-Text Label 2200 2400 2    50   ~ 0
-signal2
-Text Label 2200 2200 2    50   ~ 0
-signal1
-Text Label 3000 2800 0    50   ~ 0
-pair3-
-Text Label 3000 2700 0    50   ~ 0
-pair3+
-Text Label 3000 2500 0    50   ~ 0
-pair2-
-Text Label 3000 2400 0    50   ~ 0
-pair2+
-Text Label 3000 2200 0    50   ~ 0
-pair1-
-Text Label 3000 2100 0    50   ~ 0
-pair1+
-Text Label 3000 1900 0    50   ~ 0
-pair4-
-Text Label 3000 1800 0    50   ~ 0
 pair4+
 Text Label 8200 2000 0    50   ~ 0
@@
 pair4+
 NoConn ~ 5800 3000
-NoConn ~ 4200 3000
 NoConn ~ 7000 1700
 $Comp
-L power:GND #PWR?
+L power:GND #PWR02
 U 1 1 5C1CFAD7
 P 7600 3200
-F 0 "#PWR?" H 7600 2950 50  0001 C CNN
+F 0 "#PWR02" H 7600 2950 50  0001 C CNN
 F 1 "GND" H 7605 3027 50  0000 C CNN
 F 2 "" H 7600 3200 50  0001 C CNN
@@
 $EndComp
 $Comp
-L power:GND #PWR?
-U 1 1 5C1D03B5
-P 2600 3100
-F 0 "#PWR?" H 2600 2850 50  0001 C CNN
-F 1 "GND" H 2605 2927 50  0000 C CNN
-F 2 "" H 2600 3100 50  0001 C CNN
-F 3 "" H 2600 3100 50  0001 C CNN
-	1    2600 3100
-	1    0    0    -1
-$EndComp
-$Comp
-L power:+3.3V #PWR?
-U 1 1 5C1D1BA0
-P 2600 1500
-F 0 "#PWR?" H 2600 1350 50  0001 C CNN
-F 1 "+3.3V" H 2615 1673 50  0000 C CNN
-F 2 "" H 2600 1500 50  0001 C CNN
-F 3 "" H 2600 1500 50  0001 C CNN
-	1    2600 1500
-	1    0    0    -1
-$EndComp
-$Comp
-L power:+3.3V #PWR?
+L power:+3.3V #PWR01
 U 1 1 5C1D2224
 P 7600 1400
-F 0 "#PWR?" H 7600 1250 50  0001 C CNN
+F 0 "#PWR01" H 7600 1250 50  0001 C CNN
 F 1 "+3.3V" H 7615 1573 50  0000 C CNN
 F 2 "" H 7600 1400 50  0001 C CNN
@@
 $EndComp
 $Comp
-L Device:C C?
-U 1 1 5C1D77E3
-P 1950 1150
-F 0 "C?" H 2065 1196 50  0000 L CNN
-F 1 "0.1uF" H 2065 1105 50  0000 L CNN
-F 2 "Capacitor_SMD:C_0603_1608Metric_Pad1.05x0.95mm_HandSolder" H 1988 1000 50  0001 C CNN
-F 3 "~" H 1950 1150 50  0001 C CNN
-	1    1950 1150
-	1    0    0    -1
-$EndComp
-$Comp
-L power:+3.3V #PWR?
-U 1 1 5C1D8AC0
-P 1950 1000
-F 0 "#PWR?" H 1950 850 50  0001 C CNN
-F 1 "+3.3V" H 1965 1173 50  0000 C CNN
-F 2 "" H 1950 1000 50  0001 C CNN
-F 3 "" H 1950 1000 50  0001 C CNN
-	1    1950 1000
-	1    0    0    -1
-$EndComp
-$Comp
-L power:GND #PWR?
-U 1 1 5C1D9027
-P 1950 1300
-F 0 "#PWR?" H 1950 1050 50  0001 C CNN
-F 1 "GND" H 1955 1127 50  0000 C CNN
-F 2 "" H 1950 1300 50  0001 C CNN
-F 3 "" H 1950 1300 50  0001 C CNN
-	1    1950 1300
-	1    0    0    -1
-$EndComp
-$Comp
-L Device:C C?
+L Device:C C1
 U 1 1 5C1DA101
 P 8350 1100
-F 0 "C?" H 8465 1146 50  0000 L CNN
+F 0 "C1" H 8465 1146 50  0000 L CNN
 F 1 "0.1uF" H 8465 1055 50  0000 L CNN
 F 2 "Capacitor_SMD:C_0603_1608Metric_Pad1.05x0.95mm_HandSolder" H 8388 950 50  0001 C CNN
@@
 $EndComp
 $Comp
-L power:+3.3V #PWR?
+L power:+3.3V #PWR03
 U 1 1 5C1DA10B
 P 8350 950
-F 0 "#PWR?" H 8350 800 50  0001 C CNN
+F 0 "#PWR03" H 8350 800 50  0001 C CNN
 F 1 "+3.3V" H 8365 1123 50  0000 C CNN
 F 2 "" H 8350 950 50  0001 C CNN
@@
 $EndComp
 $Comp
-L power:GND #PWR?
+L power:GND #PWR04
 U 1 1 5C1DA115
 P 8350 1250
-F 0 "#PWR?" H 8350 1000 50  0001 C CNN
+F 0 "#PWR04" H 8350 1000 50  0001 C CNN
 F 1 "GND" H 8355 1077 50  0000 C CNN
 F 2 "" H 8350 1250 50  0001 C CNN
@@
 Text Label 7000 1600 2    50   ~ 0
 EN
-Text Label 2200 2000 2    50   ~ 0
-EN
-Text Label 2200 2600 2    50   ~ 0
-EN
-$Comp
-L Connector_Generic:Conn_01x06 J?
-U 1 1 5C1E3650
-P 1000 2200
-F 0 "J?" H 1000 2500 50  0000 C CNN
-F 1 "signal_in" V 1100 2150 50  0000 C CNN
-F 2 "" H 1000 2200 50  0001 C CNN
-F 3 "~" H 1000 2200 50  0001 C CNN
-	1    1000 2200
-	-1   0    0    -1
-$EndComp
-Text Label 1200 2400 0    50   ~ 0
-signal4
-Text Label 1200 2300 0    50   ~ 0
-signal3
-Text Label 1200 2200 0    50   ~ 0
-signal2
-Text Label 1200 2100 0    50   ~ 0
-signal1
-$Comp
-L power:GND #PWR?
-U 1 1 5C21F91E
-P 1200 2500
-F 0 "#PWR?" H 1200 2250 50  0001 C CNN
-F 1 "GND" H 1205 2327 50  0000 C CNN
-F 2 "" H 1200 2500 50  0001 C CNN
-F 3 "" H 1200 2500 50  0001 C CNN
-	1    1200 2500
-	1    0    0    -1
-$EndComp
-$Comp
-L power:+3.3V #PWR?
-U 1 1 5C21FC04
-P 1200 2000
-F 0 "#PWR?" H 1200 1850 50  0001 C CNN
-F 1 "+3.3V" H 1215 2173 50  0000 C CNN
-F 2 "" H 1200 2000 50  0001 C CNN
-F 3 "" H 1200 2000 50  0001 C CNN
-	1    1200 2000
-	1    0    0    -1
-$EndComp
-$Comp
-L Connector_Generic:Conn_01x06 J?
+$Comp
+L Connector_Generic:Conn_01x06 J2
 U 1 1 5C221C21
 P 9500 2200
-F 0 "J?" H 9500 2500 50  0000 C CNN
+F 0 "J2" H 9500 2500 50  0000 C CNN
 F 1 "signal_out" V 9600 2150 50  0000 C CNN
-F 2 "" H 9500 2200 50  0001 C CNN
+F 2 "Connector_PinHeader_2.54mm:PinHeader_1x06_P2.54mm_Horizontal" H 9500 2200 50  0001 C CNN
 F 3 "~" H 9500 2200 50  0001 C CNN
 	1    9500 2200
@@
 signal1
 $Comp
-L power:GND #PWR?
+L power:GND #PWR06
 U 1 1 5C221C2F
 P 9300 2500
-F 0 "#PWR?" H 9300 2250 50  0001 C CNN
+F 0 "#PWR06" H 9300 2250 50  0001 C CNN
 F 1 "GND" H 9305 2327 50  0000 C CNN
 F 2 "" H 9300 2500 50  0001 C CNN
@@
 $EndComp
 $Comp
-L power:+3.3V #PWR?
+L power:+3.3V #PWR05
 U 1 1 5C221C39
 P 9300 2000
-F 0 "#PWR?" H 9300 1850 50  0001 C CNN
+F 0 "#PWR05" H 9300 1850 50  0001 C CNN
 F 1 "+3.3V" H 9315 2173 50  0000 C CNN
 F 2 "" H 9300 2000 50  0001 C CNN
@@
 	-1   0    0    -1
 $EndComp
+$Comp
+L power:PWR_FLAG #FLG0101
+U 1 1 5C138695
+P 8950 2000
+F 0 "#FLG0101" H 8950 2075 50  0001 C CNN
+F 1 "PWR_FLAG" H 8950 2173 50  0000 C CNN
+F 2 "" H 8950 2000 50  0001 C CNN
+F 3 "~" H 8950 2000 50  0001 C CNN
+	1    8950 2000
+	1    0    0    -1
+$EndComp
+Wire Wire Line
+	8950 2000 9300 2000
+Connection ~ 9300 2000
+$Comp
+L power:+3.3V #PWR0101
+U 1 1 5C13D627
+P 6800 1300
+F 0 "#PWR0101" H 6800 1150 50  0001 C CNN
+F 1 "+3.3V" H 6815 1473 50  0000 C CNN
+F 2 "" H 6800 1300 50  0001 C CNN
+F 3 "" H 6800 1300 50  0001 C CNN
+	1    6800 1300
+	1    0    0    -1
+$EndComp
+$Comp
+L Device:R R1
+U 1 1 5C13DB8A
+P 6800 1450
+F 0 "R1" H 6870 1496 50  0000 L CNN
+F 1 "10k" H 6870 1405 50  0000 L CNN
+F 2 "Resistor_SMD:R_1206_3216Metric_Pad1.42x1.75mm_HandSolder" V 6730 1450 50  0001 C CNN
+F 3 "~" H 6800 1450 50  0001 C CNN
+	1    6800 1450
+	1    0    0    -1
+$EndComp
+Wire Wire Line
+	6800 1600 7000 1600
+$Comp
+L power:PWR_FLAG #FLG0102
+U 1 1 5C142446
+P 9000 2500
+F 0 "#FLG0102" H 9000 2575 50  0001 C CNN
+F 1 "PWR_FLAG" H 9000 2673 50  0000 C CNN
+F 2 "" H 9000 2500 50  0001 C CNN
+F 3 "~" H 9000 2500 50  0001 C CNN
+	1    9000 2500
+	-1   0    0    1
+$EndComp
+Wire Wire Line
+	9000 2500 9300 2500
+Connection ~ 9300 2500
 $EndSCHEMATC

Commit message: exported..
Parts:
- J2: renamed from J1; footprint Connector_RJ:RJ45_Amphenol_RJHSE5380 -> Connector_RJ:RJ45_Stewart_SS-6488S-A-NF
- renumbered J2 to J1
Connections:
- net +3V3: now also J1.6 (Pin_6); no longer J1.1 (Pin_1)
- net GND: now also J1.1 (Pin_1); no longer J1.6 (Pin_6)
- net pair1+: now also U1.6 (RIN3+); no longer U1.3 (RIN2+)
- net pair1-: now also U1.5 (RIN3-); no longer U1.4 (RIN2-)
- net pair2+: now also U1.3 (RIN2+); no longer U1.6 (RIN3+)
- net pair2-: now also U1.4 (RIN2-); no longer U1.5 (RIN3-)
- net pair3+: now also U1.2 (RIN1+); no longer U1.7 (RIN4+)
- net pair3-: now also U1.1 (RIN1-); no longer U1.8 (RIN4-)
- net pair4+: now also U1.7 (RIN4+); no longer U1.2 (RIN1+)
- net pair4-: now also U1.8 (RIN4-); no longer U1.1 (RIN1-)
- net signal1: now also J1.4 (Pin_4), U1.11 (ROUT3); no longer J1.2 (Pin_2), U1.14 (ROUT2)
- net signal2: now also U1.14 (ROUT2); no longer U1.11 (ROUT3)
- net signal3: now also J1.2 (Pin_2), U1.15 (ROUT1); no longer J1.4 (Pin_4), U1.10 (ROUT4)
- net signal4: now also U1.10 (ROUT4); no longer U1.15 (ROUT1)
Other:
- moved on the sheet: J1
Changed lines of the file:
@@
 $EndComp
 $Comp
-L Connector:8P8C_Shielded J1
+L Connector:8P8C_Shielded J2
 U 1 1 5C15786C
 P 5800 2500
-F 0 "J1" H 5857 3167 50  0000 C CNN
+F 0 "J2" H 5857 3167 50  0000 C CNN
 F 1 "LVDS_input" H 5857 3076 50  0000 C CNN
-F 2 "Connector_RJ:RJ45_Amphenol_RJHSE5380" V 5800 2525 50  0001 C CNN
+F 2 "Connector_RJ:RJ45_Stewart_SS-6488S-A-NF" V 5800 2525 50  0001 C CNN
 F 3 "~" V 5800 2525 50  0001 C CNN
 	1    5800 2500
@@
 Text Label 6200 2100 0    50   ~ 0
 pair4+
+Text Label 8200 2900 0    50   ~ 0
+signal4
 Text Label 8200 2000 0    50   ~ 0
-signal4
-Text Label 8200 2900 0    50   ~ 0
 signal3
+Text Label 8200 2300 0    50   ~ 0
+signal2
 Text Label 8200 2600 0    50   ~ 0
-signal2
-Text Label 8200 2300 0    50   ~ 0
 signal1
+Text Label 7000 1900 2    50   ~ 0
+pair3-
+Text Label 7000 2000 2    50   ~ 0
+pair3+
+Text Label 7000 2200 2    50   ~ 0
+pair2-
+Text Label 7000 2300 2    50   ~ 0
+pair2+
+Text Label 7000 2500 2    50   ~ 0
+pair1-
+Text Label 7000 2600 2    50   ~ 0
+pair1+
 Text Label 7000 2800 2    50   ~ 0
-pair3-
+pair4-
 Text Label 7000 2900 2    50   ~ 0
-pair3+
-Text Label 7000 2500 2    50   ~ 0
-pair2-
-Text Label 7000 2600 2    50   ~ 0
-pair2+
-Text Label 7000 2200 2    50   ~ 0
-pair1-
-Text Label 7000 2300 2    50   ~ 0
-pair1+
-Text Label 7000 1900 2    50   ~ 0
-pair4-
-Text Label 7000 2000 2    50   ~ 0
 pair4+
 NoConn ~ 5800 3000
@@
 EN
 $Comp
-L Connector_Generic:Conn_01x06 J2
+L Connector_Generic:Conn_01x06 J1
 U 1 1 5C221C21
-P 9500 2200
-F 0 "J2" H 9500 2500 50  0000 C CNN
-F 1 "signal_out" V 9600 2150 50  0000 C CNN
-F 2 "Connector_PinHeader_2.54mm:PinHeader_1x06_P2.54mm_Horizontal" H 9500 2200 50  0001 C CNN
-F 3 "~" H 9500 2200 50  0001 C CNN
-	1    9500 2200
-	1    0    0    -1
-$EndComp
-Text Label 9300 2400 2    50   ~ 0
+P 9500 2250
+F 0 "J1" H 9500 2550 50  0000 C CNN
+F 1 "signal_out" V 9600 2200 50  0000 C CNN
+F 2 "Connector_PinHeader_2.54mm:PinHeader_1x06_P2.54mm_Horizontal" H 9500 2250 50  0001 C CNN
+F 3 "~" H 9500 2250 50  0001 C CNN
+	1    9500 2250
+	1    0    0    1
+$EndComp
+Text Label 9300 2050 2    50   ~ 0
 signal4
-Text Label 9300 2300 2    50   ~ 0
+Text Label 9300 2350 2    50   ~ 0
 signal3
-Text Label 9300 2200 2    50   ~ 0
+Text Label 9300 2250 2    50   ~ 0
 signal2
-Text Label 9300 2100 2    50   ~ 0
+Text Label 9300 2150 2    50   ~ 0
 signal1
 $Comp
 L power:GND #PWR06
 U 1 1 5C221C2F
-P 9300 2500
-F 0 "#PWR06" H 9300 2250 50  0001 C CNN
-F 1 "GND" H 9305 2327 50  0000 C CNN
-F 2 "" H 9300 2500 50  0001 C CNN
-F 3 "" H 9300 2500 50  0001 C CNN
-	1    9300 2500
+P 9300 2450
+F 0 "#PWR06" H 9300 2200 50  0001 C CNN
+F 1 "GND" H 9305 2277 50  0000 C CNN
+F 2 "" H 9300 2450 50  0001 C CNN
+F 3 "" H 9300 2450 50  0001 C CNN
+	1    9300 2450
 	-1   0    0    -1
 $EndComp
@@
 L power:+3.3V #PWR05
 U 1 1 5C221C39
-P 9300 2000
-F 0 "#PWR05" H 9300 1850 50  0001 C CNN
-F 1 "+3.3V" H 9315 2173 50  0000 C CNN
-F 2 "" H 9300 2000 50  0001 C CNN
-F 3 "" H 9300 2000 50  0001 C CNN
-	1    9300 2000
+P 9300 1950
+F 0 "#PWR05" H 9300 1800 50  0001 C CNN
+F 1 "+3.3V" H 9315 2123 50  0000 C CNN
+F 2 "" H 9300 1950 50  0001 C CNN
+F 3 "" H 9300 1950 50  0001 C CNN
+	1    9300 1950
 	-1   0    0    -1
 $EndComp
@@
 L power:PWR_FLAG #FLG0101
 U 1 1 5C138695
-P 8950 2000
-F 0 "#FLG0101" H 8950 2075 50  0001 C CNN
-F 1 "PWR_FLAG" H 8950 2173 50  0000 C CNN
-F 2 "" H 8950 2000 50  0001 C CNN
-F 3 "~" H 8950 2000 50  0001 C CNN
-	1    8950 2000
-	1    0    0    -1
+P 8950 2450
+F 0 "#FLG0101" H 8950 2525 50  0001 C CNN
+F 1 "PWR_FLAG" H 8950 2623 50  0000 C CNN
+F 2 "" H 8950 2450 50  0001 C CNN
+F 3 "~" H 8950 2450 50  0001 C CNN
+	1    8950 2450
+	1    0    0    1
 $EndComp
 Wire Wire Line
-	8950 2000 9300 2000
-Connection ~ 9300 2000
+	8950 2450 9300 2450
 $Comp
 L power:+3.3V #PWR0101
@@
 L power:PWR_FLAG #FLG0102
 U 1 1 5C142446
-P 9000 2500
-F 0 "#FLG0102" H 9000 2575 50  0001 C CNN
-F 1 "PWR_FLAG" H 9000 2673 50  0000 C CNN
-F 2 "" H 9000 2500 50  0001 C CNN
-F 3 "~" H 9000 2500 50  0001 C CNN
-	1    9000 2500
-	-1   0    0    1
+P 8950 1950
+F 0 "#FLG0102" H 8950 2025 50  0001 C CNN
+F 1 "PWR_FLAG" H 8950 2123 50  0000 C CNN
+F 2 "" H 8950 1950 50  0001 C CNN
+F 3 "~" H 8950 1950 50  0001 C CNN
+	1    8950 1950
+	-1   0    0    -1
 $EndComp
 Wire Wire Line
-	9000 2500 9300 2500
-Connection ~ 9300 2500
+	8950 1950 9300 1950
+Connection ~ 9300 1950
+Connection ~ 9300 2450
 $EndSCHEMATC
